Commit message: changed variable names and included backup

File: robots/iCub/robots/model_backup.urdf (robot description, URDF)
Before this commit: robot iCub, 102 links, 101 joints
Links:
- removed link l_ail3
- removed link l_hand_base_link
- removed link l_lil3
- removed link l_ml3
- removed link l_ril3
- removed link l_tl4
- removed link r_ail3
- removed link r_hand_base_link
- removed link r_lil3
- removed link r_ml3
- removed link r_ril3
- removed link r_tl4
- added link l_hand, mass 0.247806; collision mesh filename=package://iCub/meshes/col_LeftHandPalm.dae scale=1.0 1.0 1.0; visual mesh filename=package://iCub/meshes/full_LeftHandPalm.dae scale=1.0 1.0 1.0
- added link l_hand_index_3, mass 0.01; collision mesh filename=package://iCub/meshes/col_LeftIndex3.dae scale=1.0 1.0 1.0; visual mesh filename=package://iCub/meshes/full_LeftIndex3.dae scale=1.0 1.0 1.0
- added link l_hand_little_3, mass 0.01; collision mesh filename=package://iCub/meshes/col_LeftLittle3.dae scale=1.0 1.0 1.0; visual mesh filename=package://iCub/meshes/full_LeftLittle3.dae scale=1.0 1.0 1.0
- added link l_hand_middle_3, mass 0.01; collision mesh filename=package://iCub/meshes/col_LeftMiddle3.dae scale=1.0 1.0 1.0; visual mesh filename=package://iCub/meshes/full_LeftMiddle3.dae scale=1.0 1.0 1.0
- added link l_hand_ring_3, mass 0.01; collision mesh filename=package://iCub/meshes/col_LeftRing3.dae scale=1.0 1.0 1.0; visual mesh filename=package://iCub/meshes/full_LeftRing3.dae scale=1.0 1.0 1.0
- added link l_hand_thumb_3, mass 0.01; collision mesh filename=package://iCub/meshes/col_LeftThumb3.dae scale=1.0 1.0 1.0; visual mesh filename=package://iCub/meshes/full_LeftThumb3.dae scale=1.0 1.0 1.0
- added link r_hand, mass 0.248289; collision mesh filename=package://iCub/meshes/col_RightHandPalm.dae scale=1.0 1.0 1.0; visual mesh filename=package://iCub/meshes/full_RightHandPalm.dae scale=1.0 1.0 1.0
- added link r_hand_index_3, mass 0.01; collision mesh filename=package://iCub/meshes/col_RightIndex3.dae scale=1.0 1.0 1.0; visual mesh filename=package://iCub/meshes/full_RightIndex3.dae scale=1.0 1.0 1.0
- added link r_hand_little_3, mass 0.01; collision mesh filename=package://iCub/meshes/col_RightLittle3.dae scale=1.0 1.0 1.0; visual mesh filename=package://iCub/meshes/full_RightLittle3.dae scale=1.0 1.0 1.0
- added link r_hand_middle_3, mass 0.01; collision mesh filename=package://iCub/meshes/col_RightMiddle3.dae scale=1.0 1.0 1.0; visual mesh filename=package://iCub/meshes/full_RightMiddle3.dae scale=1.0 1.0 1.0
- added link r_hand_ring_3, mass 0.01; collision mesh filename=package://iCub/meshes/col_RightRing3.dae scale=1.0 1.0 1.0; visual mesh filename=package://iCub/meshes/full_RightRing3.dae scale=1.0 1.0 1.0
- added link r_hand_thumb_3, mass 0.01; collision mesh filename=package://iCub/meshes/col_RightThumb3.dae scale=1.0 1.0 1.0; visual mesh filename=package://iCub/meshes/full_RightThumb3.dae scale=1.0 1.0 1.0
Joints:
- joint l_hand_dh_frame_fixed_joint: parent l_hand_base_link -> l_hand
- joint l_hand_index_0_joint: parent l_hand_base_link -> l_hand
- joint l_hand_index_3_joint: child l_ail3 -> l_hand_index_3
- joint l_hand_index_tip_joint: parent l_ail3 -> l_hand_index_3
- joint l_hand_little_0_joint: parent l_hand_base_link -> l_hand
- joint l_hand_little_3_joint: child l_lil3 -> l_hand_little_3
- joint l_hand_little_tip_joint: parent l_lil3 -> l_hand_little_3
- joint l_hand_middle_0_joint: parent l_hand_base_link -> l_hand
- joint l_hand_middle_3_joint: child l_ml3 -> l_hand_middle_3
- joint l_hand_middle_tip_joint: parent l_ml3 -> l_hand_middle_3
- joint l_hand_ring_0_joint: parent l_hand_base_link -> l_hand
- joint l_hand_ring_3_joint: child l_ril3 -> l_hand_ring_3
- joint l_hand_ring_tip_joint: parent l_ril3 -> l_hand_ring_3
- joint l_hand_thumb_0_joint: parent l_hand_base_link -> l_hand
- joint l_hand_thumb_3_joint: child l_tl4 -> l_hand_thumb_3
- joint l_hand_thumb_tip_joint: parent l_tl4 -> l_hand_thumb_3
- joint l_wrist_yaw: child l_hand_base_link -> l_hand
- joint r_hand_dh_frame_fixed_joint: parent r_hand_base_link -> r_hand
- joint r_hand_index_0_joint: parent r_hand_base_link -> r_hand
- joint r_hand_index_3_joint: child r_ail3 -> r_hand_index_3
- joint r_hand_index_tip_joint: parent r_ail3 -> r_hand_index_3
- joint r_hand_little_0_joint: parent r_hand_base_link -> r_hand
- joint r_hand_little_3_joint: child r_lil3 -> r_hand_little_3
- joint r_hand_little_tip_joint: parent r_lil3s -> r_hand_little_3
- joint r_hand_middle_0_joint: parent r_hand_base_link -> r_hand
- joint r_hand_middle_3_joint: child r_ml3 -> r_hand_middle_3
- joint r_hand_middle_tip_joint: parent r_ml3 -> r_hand_middle_3
- joint r_hand_ring_0_joint: parent r_hand_base_link -> r_hand
- joint r_hand_ring_3_joint: child r_ril3 -> r_hand_ring_3
- joint r_hand_ring_tip_joint: parent r_ril3 -> r_hand_ring_3
- joint r_hand_thumb_0_joint: parent r_hand_base_link -> r_hand
- joint r_hand_thumb_3_joint: child r_tl4 -> r_hand_thumb_3
- joint r_hand_thumb_tip_joint: parent r_tl4 -> r_hand_thumb_3
- joint r_wrist_yaw: child r_hand_base_link -> r_hand
